File: MacClassicRAMCard.kicad_pcb (KiCad board)
At the start: 2 copper layers, 58.4 x 38.7 mm, 19 parts, among them J1 RAM Exp., U1 AS4C1M16F5, U2 AS4C1M16F5, U3 74LS08

Commit message: Finished layout I think
Parts:
- removed the C1 at (146.1, 95.5)
- added C6: 2u2, stdpads:C_0805, F.Cu at (115.6, 95.5)
- added FID3: Fiducial, stdpads:Fiducial, F.Cu at (145.8, 133.3)
- added FID4: Fiducial, stdpads:Fiducial, F.Cu at (95.5, 133.3)
- added H1: , stdpads:PasteHole_1.1mm_PTH, F.Cu at (148.3, 133.3)
- added H4: , stdpads:PasteHole_1.1mm_PTH, F.Cu at (93.0, 133.3)
- U1, U2: footprint stdpads:SOJ-42-400mil-Skinny -> stdpads:SOJ-42_400mil
- moved C7 48.6 mm to (146.1, 95.5)
- moved C3 48.4 mm to (98.4, 111.5), turned to 270 degrees
- moved C2 39.3 mm to (146.1, 120.3), turned to 0 degrees
- moved U3 6.35 mm to (104.1, 113.0)
- renumbered C3 to C1, C5 to C4, C4 to C5
Connections:
- U1 pad 10: /DQ7 -> /DQ4
- U1 pad 15: (no net) -> Net-(U1-Pad15)
- U1 pad 16: (no net) -> Net-(U1-Pad16)
- U1 pad 2: /DQ0 -> /DQ3
- U1 pad 3: /DQ1 -> /DQ7
- U1 pad 33: /DQ8 -> /DQ10
- U1 pad 34: /DQ9 -> /DQ8
- U1 pad 35: /DQ10 -> /DQ11
- U1 pad 36: /DQ11 -> /DQ9
- U1 pad 38: /DQ12 -> /DQ14
- U1 pad 39: /DQ13 -> /DQ12
- U1 pad 40: /DQ14 -> /DQ15
- U1 pad 41: /DQ15 -> /DQ13
- U1 pad 5: /DQ3 -> /DQ6
- U1 pad 7: /DQ4 -> /DQ1
- U1 pad 9: /DQ6 -> /DQ0
- U2 pad 10: /DQ7 -> /DQ4
- U2 pad 15: (no net) -> Net-(U2-Pad15)
- U2 pad 16: (no net) -> Net-(U2-Pad16)
- U2 pad 2: /DQ0 -> /DQ3
- U2 pad 3: /DQ1 -> /DQ7
- U2 pad 33: /DQ8 -> /DQ10
- U2 pad 34: /DQ9 -> /DQ8
- U2 pad 35: /DQ10 -> /DQ11
- U2 pad 36: /DQ11 -> /DQ9
- U2 pad 38: /DQ12 -> /DQ14
- U2 pad 39: /DQ13 -> /DQ12
- U2 pad 40: /DQ14 -> /DQ15
- U2 pad 41: /DQ15 -> /DQ13
- U2 pad 5: /DQ3 -> /DQ6
- U2 pad 7: /DQ4 -> /DQ1
- U2 pad 9: /DQ6 -> /DQ0
Routing:
- net +5V: track 605.4 -> 713.0 mm, vias 33 -> 34
- net /L~CAS~1: track 58.4 -> 92.7 mm
- net /U~CAS~1: track 50.3 -> 83.3 mm, vias 0 -> 1
- net /~OE~1: track 37.1 -> 69.3 mm
- net /DQ0: track 19.9 -> 50.4 mm
- net /DQ1: track 19.9 -> 50.4 mm
- net /U~CAS~0: track 35.2 -> 61.1 mm
- net /L~CAS~0: track 45.0 -> 66.8 mm, vias 0 -> 2
- net /~OE~0: track 24.5 -> 46.2 mm
- net /DQ3: track 73.3 -> 51.7 mm
- net /DQ7: track 66.8 -> 48.3 mm
- net /DQ9: track 22.8 -> 34.1 mm
- net /DQ11: track 20.7 -> 30.7 mm
- net /DQ8: track 25.6 -> 34.1 mm
- net /~RAS~: track 47.3 -> 40.1 mm
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Other:
- board size 58.4 x 38.7 mm -> 58.4 x 46 mm
