File: MacClassicRAMCard.kicad_pcb (KiCad board)
At the start: 2 copper layers, 68.6 x 46 mm, 19 parts, among them J1 RAM Exp., U1 AS4C1M16F5, U2 AS4C1M16F5, U3 74HCT08D

Commit message: New prototype
Parts:
- added H5: , stdpads:PasteHole_1.152mm_NPTH, F.Cu at (153.4, 133.3)
- added H6: , stdpads:PasteHole_1.152mm_NPTH, F.Cu at (87.9, 133.3)
- added H7: , stdpads:PasteHole_1.152mm_NPTH, F.Cu at (90.4, 90.4)
- moved FID4 2.54 mm to (93.0, 90.4)
Connections:
- J1 pad 10: /U~{CAS}D -> /L~{CAS}D
- J1 pad 35: /~{WE} -> /~{RAS}
- J1 pad 36: /~{RAS} -> /~{WE}
- J1 pad 5: /L~{CAS}C -> /U~{CAS}C
- J1 pad 6: /U~{CAS}C -> /L~{CAS}C
- J1 pad 7: /U~{CAS}1 -> /L~{CAS}1
- J1 pad 8: /L~{CAS}1 -> /U~{CAS}1
- J1 pad 9: /L~{CAS}D -> /U~{CAS}D
- U1 pad 11: Net-(U1-Pad11) -> unconnected-(U1-Pad11)
- U1 pad 12: Net-(U1-Pad12) -> unconnected-(U1-Pad12)
- U1 pad 15: Net-(U1-Pad15) -> unconnected-(U1-Pad15)
- U1 pad 16: Net-(U1-Pad16) -> unconnected-(U1-Pad16)
- U1 pad 32: Net-(U1-Pad32) -> unconnected-(U1-Pad32)
- U2 pad 11: Net-(U2-Pad11) -> unconnected-(U2-Pad11)
- U2 pad 12: Net-(U2-Pad12) -> unconnected-(U2-Pad12)
- U2 pad 15: Net-(U2-Pad15) -> unconnected-(U2-Pad15)
- U2 pad 16: Net-(U2-Pad16) -> unconnected-(U2-Pad16)
- U2 pad 32: Net-(U2-Pad32) -> unconnected-(U2-Pad32)
- U3 pad 1: /L~{CAS}C -> /U~{CAS}C
- U3 pad 10: /L~{CAS}0 -> /U~{CAS}0
- U3 pad 12: /U~{CAS}1 -> /L~{CAS}1
- U3 pad 13: /L~{CAS}1 -> /U~{CAS}1
- U3 pad 2: /L~{CAS}D -> /U~{CAS}D
- U3 pad 3: /L~{CAS}0 -> /U~{CAS}0
- U3 pad 4: /U~{CAS}C -> /L~{CAS}C
- U3 pad 5: /U~{CAS}D -> /L~{CAS}D
- U3 pad 6: /U~{CAS}0 -> /L~{CAS}0
- U3 pad 9: /U~{CAS}0 -> /L~{CAS}0
Routing:
- net /~{WE}: track 36.7 -> 41.4 mm
- net /U~{CAS}C: track 12.3 -> 8.21 mm, vias 1 -> 0
- net /L~{CAS}C: track 8.21 -> 12.3 mm, vias 0 -> 1
- net /U~{CAS}1: track 83.3 -> 87.3 mm, vias 1 -> 0
- net /L~{CAS}1: track 92.7 -> 89.6 mm, vias 2 -> 5
- net /U~{CAS}0: track 61.1 -> 64.1 mm, vias 0 -> 2
- net /~{RAS}: track 40.1 -> 38.0 mm
- net /L~{CAS}0: track 66.8 -> 64.7 mm
- net /U~{CAS}D: track 10.8 -> 8.74 mm
- net /L~{CAS}D: track 8.74 -> 10.8 mm
- net +5V: vias 35 -> 33
- net GND: vias 176 -> 198
Other:
- board text added: "0.2"

Commit message: New logo
Parts:
- added G***: LOGO, LOGO, F.Cu at (98.6, 96.3)
- added G***: LOGO, LOGO, F.Cu at (98.6, 102.2)
- added H8: , stdpads:PasteHole_3mm_NPTH, F.Cu at (147.8, 91.3)
- added H9: , stdpads:PasteHole_3mm_NPTH, F.Cu at (93.5, 91.3)
- moved H7 3.59 mm to (87.9, 93.0)
- moved FID4 2.54 mm to (90.4, 90.4)
Routing:
- net GND: vias 198 -> 283
Other:
- board text added: "JLCJLCJLCJLC"
- board text removed: "0.2"
- board text removed: "3 MB RAM"
- board text removed: "4406A"
- board text removed: "GW"
- board text removed: "Garrett’s Workshop"
- board text removed: "JLCJLCJLC"
- board text removed: "for Macintosh Classic"
