File: MacClassicRAMCard-tall.kicad_pcb (KiCad board)
At the start: 2 copper layers, 58.4 x 46 mm, 23 parts, among them J1 RAM Exp., U1 AS4C1M16F5, U2 AS4C1M16F5, U3 74HCT08D

Commit message: As sent to JLC
Parts:
- removed the FID1 at (93.0, 118.4)
- removed the FID2 at (148.3, 118.4)
- moved FID4 7.18 mm to (150.9, 85.3)
- moved FID3 7.18 mm to (90.4, 85.3)
- moved H1 7.18 mm to (87.9, 85.3)
- moved H4 7.18 mm to (153.4, 85.3)
- moved H2 6.43 mm to (87.9, 119.8)
- moved H3 6.43 mm to (153.4, 119.8)
- moved FID1 2.54 mm to (94.2, 133.3)
- moved FID2 2.54 mm to (147.1, 133.3)
- moved H5 2.54 mm to (94.2, 130.8)
- moved H6 2.54 mm to (147.1, 130.8)
- renumbered FID5 to FID1, FID6 to FID2
Routing:
- net GND: vias 162 -> 167
Other:
- board size 58.4 x 46 mm -> 68.6 x 51.1 mm
