File: MacClassicRAMCard.sch (KiCad schematic (older format))
At the start: 19 parts, among them J1 RAM Exp., U1 AS4C1M16F5, U2 AS4C1M16F5, U3 74LS08

Commit message: Finished layout I think
Parts:
- U1, U2: footprint stdpads:SOJ-42-400mil-Skinny -> stdpads:SOJ-42_400mil
Connections:
- net DQ0: now also U1.9 (DQ6), U2.9 (DQ6); no longer U1.2 (DQ0), U2.2 (DQ0)
- net DQ1: now also U1.7 (DQ4), U2.7 (DQ4); no longer U1.3 (DQ1), U2.3 (DQ1)
- net DQ10: now also U1.33 (DQ8), U2.33 (DQ8); no longer U1.35 (DQ10), U2.35 (DQ10)
- net DQ11: now also U1.35 (DQ10), U2.35 (DQ10); no longer U1.36 (DQ11), U2.36 (DQ11)
- net DQ12: now also U1.39 (DQ13), U2.39 (DQ13); no longer U1.38 (DQ12), U2.38 (DQ12)
- net DQ13: now also U1.41 (DQ15), U2.41 (DQ15); no longer U1.39 (DQ13), U2.39 (DQ13)
- net DQ14: now also U1.38 (DQ12), U2.38 (DQ12); no longer U1.40 (DQ14), U2.40 (DQ14)
- net DQ15: now also U1.40 (DQ14), U2.40 (DQ14); no longer U1.41 (DQ15), U2.41 (DQ15)
- net DQ3: now also U1.2 (DQ0), U2.2 (DQ0); no longer U1.5 (DQ3), U2.5 (DQ3)
- net DQ4: now also U1.10 (DQ7), U2.10 (DQ7); no longer U1.7 (DQ4), U2.7 (DQ4)
- net DQ6: now also U1.5 (DQ3), U2.5 (DQ3); no longer U1.9 (DQ6), U2.9 (DQ6)
- net DQ7: now also U1.3 (DQ1), U2.3 (DQ1); no longer U1.10 (DQ7), U2.10 (DQ7)
- net DQ8: now also U1.34 (DQ9), U2.34 (DQ9); no longer U1.33 (DQ8), U2.33 (DQ8)
- net DQ9: now also U1.36 (DQ11), U2.36 (DQ11); no longer U1.34 (DQ9), U2.34 (DQ9)
Changed lines of the file:
@@
 	1    0    0    -1
 $EndComp
-Text Label 6600 2750 0    50   ~ 0
-DQ4
-Text Label 6600 2850 0    50   ~ 0
-DQ5
-Text Label 6600 2950 0    50   ~ 0
-DQ6
-Text Label 6600 3050 0    50   ~ 0
-DQ7
-Text Label 6600 2650 0    50   ~ 0
-DQ3
-Text Label 6600 2450 0    50   ~ 0
-DQ1
 Text Label 5800 2450 2    50   ~ 0
 A0
@@
 Text Label 5800 3350 2    50   ~ 0
 A9
-Text Label 6600 2550 0    50   ~ 0
-DQ2
-Text Label 6600 2350 0    50   ~ 0
-DQ0
 Connection ~ 9550 6050
 $Comp
@@
 F 0 "U1" H 6200 3950 50  0000 C CNN
 F 1 "AS4C1M16F5" V 6200 3150 50  0000 C CNN
-F 2 "stdpads:SOJ-42-400mil-Skinny" H 6200 2200 50  0001 C CNN
+F 2 "stdpads:SOJ-42_400mil" H 6200 2200 50  0001 C CNN
 F 3 "" H 6200 2800 50  0001 C CNN
 	1    6200 3150
@@
 Text Label 5800 3450 2    50   ~ 0
 L~CAS~0
-Text Label 6600 3650 0    50   ~ 0
-DQ12
-Text Label 6600 3750 0    50   ~ 0
-DQ13
-Text Label 6600 3850 0    50   ~ 0
-DQ14
-Text Label 6600 3950 0    50   ~ 0
-DQ15
-Text Label 6600 3550 0    50   ~ 0
-DQ11
-Text Label 6600 3350 0    50   ~ 0
-DQ9
-Text Label 6600 3450 0    50   ~ 0
-DQ10
-Text Label 6600 3250 0    50   ~ 0
-DQ8
 $Comp
 L power:GND #PWR0101
@@
 	-1   0    0    -1
 $EndComp
-Text Label 8200 2750 0    50   ~ 0
-DQ4
-Text Label 8200 2850 0    50   ~ 0
-DQ5
-Text Label 8200 2950 0    50   ~ 0
-DQ6
-Text Label 8200 3050 0    50   ~ 0
-DQ7
-Text Label 8200 2650 0    50   ~ 0
-DQ3
-Text Label 8200 2450 0    50   ~ 0
-DQ1
 Text Label 7400 2450 2    50   ~ 0
 A0
@@
 Text Label 7400 3350 2    50   ~ 0
 A9
-Text Label 8200 2550 0    50   ~ 0
-DQ2
-Text Label 8200 2350 0    50   ~ 0
-DQ0
 $Comp
 L GW_RAM:DRAM-1Mx16-SOP-42 U2
@@
 F 0 "U2" H 7800 3950 50  0000 C CNN
 F 1 "AS4C1M16F5" V 7800 3150 50  0000 C CNN
-F 2 "stdpads:SOJ-42-400mil-Skinny" H 7800 2200 50  0001 C CNN
+F 2 "stdpads:SOJ-42_400mil" H 7800 2200 50  0001 C CNN
 F 3 "" H 7800 2800 50  0001 C CNN
 	1    7800 3150
@@
 Text Label 7400 3450 2    50   ~ 0
 L~CAS~1
-Text Label 8200 3650 0    50   ~ 0
-DQ12
-Text Label 8200 3750 0    50   ~ 0
-DQ13
-Text Label 8200 3850 0    50   ~ 0
-DQ14
-Text Label 8200 3950 0    50   ~ 0
-DQ15
-Text Label 8200 3550 0    50   ~ 0
-DQ11
 Text Label 8200 3350 0    50   ~ 0
-DQ9
-Text Label 8200 3450 0    50   ~ 0
-DQ10
-Text Label 8200 3250 0    50   ~ 0
 DQ8
 $Comp
@@
 	1    0    0    -1
 $EndComp
+Text Label 6600 2950 0    50   ~ 0
+DQ0
+Text Label 6600 2750 0    50   ~ 0
+DQ1
+Text Label 6600 2850 0    50   ~ 0
+DQ5
+Text Label 6600 3050 0    50   ~ 0
+DQ4
+Text Label 6600 2650 0    50   ~ 0
+DQ6
+Text Label 6600 2450 0    50   ~ 0
+DQ7
+Text Label 6600 2550 0    50   ~ 0
+DQ2
+Text Label 6600 2350 0    50   ~ 0
+DQ3
+Text Label 8200 2950 0    50   ~ 0
+DQ0
+Text Label 8200 2750 0    50   ~ 0
+DQ1
+Text Label 8200 2850 0    50   ~ 0
+DQ5
+Text Label 8200 3050 0    50   ~ 0
+DQ4
+Text Label 8200 2650 0    50   ~ 0
+DQ6
+Text Label 8200 2450 0    50   ~ 0
+DQ7
+Text Label 8200 2550 0    50   ~ 0
+DQ2
+Text Label 8200 2350 0    50   ~ 0
+DQ3
+Text Label 8200 3750 0    50   ~ 0
+DQ12
+Text Label 8200 3950 0    50   ~ 0
+DQ13
+Text Label 8200 3650 0    50   ~ 0
+DQ14
+Text Label 8200 3850 0    50   ~ 0
+DQ15
+Text Label 6600 3750 0    50   ~ 0
+DQ12
+Text Label 6600 3950 0    50   ~ 0
+DQ13
+Text Label 6600 3650 0    50   ~ 0
+DQ14
+Text Label 6600 3850 0    50   ~ 0
+DQ15
+Text Label 8200 3250 0    50   ~ 0
+DQ10
+Text Label 8200 3550 0    50   ~ 0
+DQ9
+Text Label 8200 3450 0    50   ~ 0
+DQ11
+Text Label 6600 3350 0    50   ~ 0
+DQ8
+Text Label 6600 3250 0    50   ~ 0
+DQ10
+Text Label 6600 3550 0    50   ~ 0
+DQ9
+Text Label 6600 3450 0    50   ~ 0
+DQ11
 $EndSCHEMATC

Commit message: As sent to JLC
Parts:
- added FID5, FID6: Fiducial, stdpads:Fiducial, symbol Mechanical:Fiducial
- added H5, H6: (no value), stdpads:PasteHole_1.1mm_PTH, symbol Mechanical:MountingHole_Pad
- J1: footprint Connector_PinSocket_2.54mm:PinSocket_2x22_P2.54mm_Horizontal -> stdpads:PinSocket_2x22_P2.54mm_Horizontal
- U3: value 74LS08 -> 74HCT08D
Connections:
- net GND: now also H5.1, H6.1
Other:
- note added: "U3A and U3B combine the /CAS signals for the two 256kx4 banks.\nU3C and U3D generate /OE signals to the DRAMs.\nOn the original Classic RAM card /OE is tied low.\nThis arrangement lets us use EDO DRAM."
- moved on the sheet: C1, C2, C3, C4, C5, C6, C7, FID1, FID2, FID3, FID4, H1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

Commit message: No actually
Parts:
- removed FID5, FID6: Fiducial, stdpads:Fiducial, symbol Mechanical:Fiducial
- removed H5, H6: (no value), stdpads:PasteHole_1.1mm_PTH, symbol Mechanical:MountingHole_Pad
Other:
- moved on the sheet: FID1, FID2, FID3, FID4, H1, H2, H3, H4
Changed lines of the file:
@@
 L Mechanical:MountingHole_Pad H3
 U 1 1 5EDC8F09
-P 2700 3400
-F 0 "H3" H 2800 3403 50  0000 L CNN
-F 1 " " H 2800 3358 50  0001 L CNN
-F 2 "stdpads:PasteHole_1.1mm_PTH" H 2700 3400 50  0001 C CNN
-F 3 "~" H 2700 3400 50  0001 C CNN
-	1    2700 3400
+P 3300 3400
+F 0 "H3" H 3400 3403 50  0000 L CNN
+F 1 " " H 3400 3358 50  0001 L CNN
+F 2 "stdpads:PasteHole_1.1mm_PTH" H 3300 3400 50  0001 C CNN
+F 3 "~" H 3300 3400 50  0001 C CNN
+	1    3300 3400
 	1    0    0    -1
 $EndComp
@@
 L Mechanical:MountingHole_Pad H4
 U 1 1 5EDC8F0F
-P 3000 3400
-F 0 "H4" H 3100 3403 50  0000 L CNN
-F 1 " " H 3100 3358 50  0001 L CNN
-F 2 "stdpads:PasteHole_1.1mm_PTH" H 3000 3400 50  0001 C CNN
-F 3 "~" H 3000 3400 50  0001 C CNN
-	1    3000 3400
+P 3600 3400
+F 0 "H4" H 3700 3403 50  0000 L CNN
+F 1 " " H 3700 3358 50  0001 L CNN
+F 2 "stdpads:PasteHole_1.1mm_PTH" H 3600 3400 50  0001 C CNN
+F 3 "~" H 3600 3400 50  0001 C CNN
+	1    3600 3400
 	1    0    0    -1
 $EndComp
@@
 L Mechanical:MountingHole_Pad H2
 U 1 1 5EE01FE6
-P 2400 3400
-F 0 "H2" H 2500 3403 50  0000 L CNN
-F 1 " " H 2500 3358 50  0001 L CNN
-F 2 "stdpads:PasteHole_1.1mm_PTH" H 2400 3400 50  0001 C CNN
-F 3 "~" H 2400 3400 50  0001 C CNN
-	1    2400 3400
+P 3000 3400
+F 0 "H2" H 3100 3403 50  0000 L CNN
+F 1 " " H 3100 3358 50  0001 L CNN
+F 2 "stdpads:PasteHole_1.1mm_PTH" H 3000 3400 50  0001 C CNN
+F 3 "~" H 3000 3400 50  0001 C CNN
+	1    3000 3400
 	1    0    0    -1
 $EndComp
@@
 L Mechanical:MountingHole_Pad H1
 U 1 1 5EE01FE0
-P 2100 3400
-F 0 "H1" H 2200 3403 50  0000 L CNN
-F 1 " " H 2200 3358 50  0001 L CNN
-F 2 "stdpads:PasteHole_1.1mm_PTH" H 2100 3400 50  0001 C CNN
-F 3 "~" H 2100 3400 50  0001 C CNN
-	1    2100 3400
+P 2700 3400
+F 0 "H1" H 2800 3403 50  0000 L CNN
+F 1 " " H 2800 3358 50  0001 L CNN
+F 2 "stdpads:PasteHole_1.1mm_PTH" H 2700 3400 50  0001 C CNN
+F 3 "~" H 2700 3400 50  0001 C CNN
+	1    2700 3400
 	1    0    0    -1
 $EndComp
@@
 L Mechanical:Fiducial FID4
 U 1 1 5EDCCFC0
+P 3100 3650
+F 0 "FID4" H 3185 3696 50  0000 L CNN
+F 1 "Fiducial" H 3185 3605 50  0000 L CNN
+F 2 "stdpads:Fiducial" H 3100 3650 50  0001 C CNN
+F 3 "~" H 3100 3650 50  0001 C CNN
+	1    3100 3650
+	1    0    0    -1
+$EndComp
+$Comp
+L Mechanical:Fiducial FID2
+U 1 1 5EDCCA31
 P 2100 3650
-F 0 "FID4" H 2185 3696 50  0000 L CNN
+F 0 "FID2" H 2185 3696 50  0000 L CNN
 F 1 "Fiducial" H 2185 3605 50  0000 L CNN
 F 2 "stdpads:Fiducial" H 2100 3650 50  0001 C CNN
@@
 $EndComp
 $Comp
-L Mechanical:Fiducial FID2
-U 1 1 5EDCCA31
-P 1100 3650
-F 0 "FID2" H 1185 3696 50  0000 L CNN
-F 1 "Fiducial" H 1185 3605 50  0000 L CNN
-F 2 "stdpads:Fiducial" H 1100 3650 50  0001 C CNN
-F 3 "~" H 1100 3650 50  0001 C CNN
-	1    1100 3650
-	1    0    0    -1
-$EndComp
-$Comp
 L Mechanical:Fiducial FID1
 U 1 1 5EDCC581
-P 1100 3400
-F 0 "FID1" H 1185 3446 50  0000 L CNN
-F 1 "Fiducial" H 1185 3355 50  0000 L CNN
-F 2 "stdpads:Fiducial" H 1100 3400 50  0001 C CNN
-F 3 "~" H 1100 3400 50  0001 C CNN
-	1    1100 3400
+P 2100 3400
+F 0 "FID1" H 2185 3446 50  0000 L CNN
+F 1 "Fiducial" H 2185 3355 50  0000 L CNN
+F 2 "stdpads:Fiducial" H 2100 3400 50  0001 C CNN
+F 3 "~" H 2100 3400 50  0001 C CNN
+	1    2100 3400
 	1    0    0    -1
 $EndComp
@@
 Text Notes 1900 1250 0    50   ~ 0
 U3A and U3B combine the /CAS signals for the two 256kx4 banks.\nU3C and U3D generate /OE signals to the DRAMs.\nOn the original Classic RAM card /OE is tied low.\nThis arrangement lets us use EDO DRAM.
-$Comp
-L Mechanical:MountingHole_Pad H5
-U 1 1 628D26D2
-P 3300 3400
-F 0 "H5" H 3400 3403 50  0000 L CNN
-F 1 " " H 3400 3358 50  0001 L CNN
-F 2 "stdpads:PasteHole_1.1mm_PTH" H 3300 3400 50  0001 C CNN
-F 3 "~" H 3300 3400 50  0001 C CNN
-	1    3300 3400
-	1    0    0    -1
-$EndComp
-$Comp
-L Mechanical:MountingHole_Pad H6
-U 1 1 628D4315
-P 3600 3400
-F 0 "H6" H 3700 3403 50  0000 L CNN
-F 1 " " H 3700 3358 50  0001 L CNN
-F 2 "stdpads:PasteHole_1.1mm_PTH" H 3600 3400 50  0001 C CNN
-F 3 "~" H 3600 3400 50  0001 C CNN
-	1    3600 3400
-	1    0    0    -1
-$EndComp
-Connection ~ 2400 3500
-Connection ~ 2700 3500
 Connection ~ 3000 3500
-Wire Wire Line
-	2400 3500 2700 3500
+Connection ~ 3300 3500
+Wire Wire Line
+	3000 3500 3300 3500
+Wire Wire Line
+	3300 3500 3600 3500
 Wire Wire Line
 	2700 3500 3000 3500
-Wire Wire Line
-	3000 3500 3300 3500
-Connection ~ 3600 3500
-Connection ~ 3300 3500
-Wire Wire Line
-	3300 3500 3600 3500
-Wire Wire Line
-	2100 3500 2400 3500
 $Comp
 L Mechanical:Fiducial FID3
 U 1 1 5EDCCCF0
-P 1600 3650
-F 0 "FID3" H 1685 3696 50  0000 L CNN
-F 1 "Fiducial" H 1685 3605 50  0000 L CNN
-F 2 "stdpads:Fiducial" H 1600 3650 50  0001 C CNN
-F 3 "~" H 1600 3650 50  0001 C CNN
-	1    1600 3650
-	1    0    0    -1
-$EndComp
-$Comp
-L Mechanical:Fiducial FID6
-U 1 1 628E0825
-P 3100 3650
-F 0 "FID6" H 3185 3696 50  0000 L CNN
-F 1 "Fiducial" H 3185 3605 50  0000 L CNN
-F 2 "stdpads:Fiducial" H 3100 3650 50  0001 C CNN
-F 3 "~" H 3100 3650 50  0001 C CNN
-	1    3100 3650
-	1    0    0    -1
-$EndComp
-$Comp
-L Mechanical:Fiducial FID5
-U 1 1 628E082B
 P 2600 3650
-F 0 "FID5" H 2685 3696 50  0000 L CNN
+F 0 "FID3" H 2685 3696 50  0000 L CNN
 F 1 "Fiducial" H 2685 3605 50  0000 L CNN
 F 2 "stdpads:Fiducial" H 2600 3650 50  0001 C CNN
@@
 	1    0    0    -1
 $EndComp
+Connection ~ 3600 3500
 $EndSCHEMATC
