File: MacClassicRAMCard.kicad_sch (KiCad schematic)
At the start: 19 parts, among them J1 RAM Exp., U1 AS4C1M16F5, U2 AS4C1M16F5, U3 74HCT08D

Commit message: New prototype
Parts:
- added H5, H6, H7: (no value), stdpads:PasteHole_1.152mm_NPTH, symbol Mechanical:MountingHole_Pad
Connections:
- net GND: now also H5.1, H6.1, H7.1
- net L~{CAS}0: now also U3.6, U3.9; no longer U3.10, U3.3
- net L~{CAS}1: now also J1.7 (Pin_7), U3.12; no longer J1.8 (Pin_8), U3.13
- net L~{CAS}C: now also J1.6 (Pin_6), U3.4; no longer J1.5 (Pin_5), U3.1
- net L~{CAS}D: now also J1.10 (Pin_10), U3.5; no longer J1.9 (Pin_9), U3.2
- net U~{CAS}0: now also U3.10, U3.3; no longer U3.6, U3.9
- net U~{CAS}1: now also J1.8 (Pin_8), U3.13; no longer J1.7 (Pin_7), U3.12
- net U~{CAS}C: now also J1.5 (Pin_5), U3.1; no longer J1.6 (Pin_6), U3.4
- net U~{CAS}D: now also J1.9 (Pin_9), U3.2; no longer J1.10 (Pin_10), U3.5
- net ~{RAS}: now also J1.35 (Pin_35); no longer J1.36 (Pin_36)
- net ~{WE}: now also J1.36 (Pin_36); no longer J1.35 (Pin_35)
Other:
- company: (none) -> Garrett's Workshop
- title: (none) -> GW4406A
- moved on the sheet: FID1, H1, H2, H3, H4, U3A, U3B

Commit message: New logo
Parts:
- added H8, H9: (no value), stdpads:PasteHole_3mm_NPTH, symbol Mechanical:MountingHole
- H5, H6, H7: symbol Mechanical:MountingHole_Pad -> Mechanical:MountingHole
Connections:
- net GND: no longer H5.1, H6.1, H7.1
Other:
- moved on the sheet: FID1, FID2, FID3, FID4, H1, H2, H3, H4, U3E
